Commit message: Caster wheel hinges ready. WIP

File: ddsr_description/urdf/ddsr.xacro (robot description, xacro)
@@ -152,3 +152,67 @@
 	</inertial>
 </link>
+<!-- ~~~~~~~~~~~~~~~~~~~~~~~ CASTER WHEEL ~~~~~~~~~~~~~~~~~~~~~~~~~~~~~~~~~~~~~~~~ -->
+<joint name="$base_2_caster_hinge_1" type="continuous" >
+	<parent link="base"/>
+	<child link="caster_hinge_1"/>
+	<origin xyz="${base_length*0.4} 0 ${-base_height*0.5-0.02}" rpy="0 0 0"/>
+	<axis xyz="0 0 1"/>
+	<limit effort="100000." velocity="${2*pi}"/>
+	<dynamics friction="0.1" damping="0.01"/>
+</joint>
+<link name="caster_hinge_1">
+	<visual>
+		<origin xyz="0 0 0" rpy="0 0 0"/>
+		<geometry>
+			<box size="0.02 0.02 0.04"/>
+		</geometry>
+		<material name="ddsr/red" />
+	</visual>
+	<collision>
+		<origin xyz="0 0 0" rpy="0 0 0"/>
+		<geometry>
+			<box size="0.02 0.02 0.04"/>
+		</geometry>
+	</collision>
+	<inertial>
+		<mass value="1" />
+		<origin xyz="0 0 0" rpy="0 0 0"/>
+		<inertia ixx="${0.083*(0.02*0.02+0.04*0.04)}"
+			ixy="0.0"
+			ixz="0.0"
+			iyy="${0.083*(0.02*0.02+0.04*0.04)}"
+			iyz="0.0"
+			izz="${0.083*(0.02*0.02+0.02*0.02)}" />
+	</inertial>
+</link>
+<joint name="$caster_hinge_1_2_caster_hinge_2" type="fixed" >
+	<parent link="caster_hinge_1"/>
+	<child link="caster_hinge_2"/>
+	<origin xyz="${-0.04*0.707*0.5} 0 ${-0.02-0.04*0.707*0.5}" rpy="0 ${0.25*pi} 0"/>
+</joint>
+<link name="caster_hinge_2">
+	<visual>
+		<origin xyz="0 0 0" rpy="0 0 0"/>
+		<geometry>
+			<box size="0.02 0.02 0.04"/>
+		</geometry>
+		<material name="ddsr/red" />
+	</visual>
+	<collision>
+		<origin xyz="0 0 0" rpy="0 0 0"/>
+		<geometry>
+			<box size="0.02 0.02 0.04"/>
+		</geometry>
+	</collision>
+	<inertial>
+		<mass value="1" />
+		<origin xyz="0 0 0" rpy="0 0 0"/>
+		<inertia ixx="${0.083*(0.02*0.02+0.04*0.04)}"
+			ixy="0.0"
+			ixz="0.0"
+			iyy="${0.083*(0.02*0.02+0.04*0.04)}"
+			iyz="0.0"
+			izz="${0.083*(0.02*0.02+0.02*0.02)}" />
+	</inertial>
+</link>
 </robot>

Commit message: First version of full xacro description, with both drive wheels and one caster wheel

File: ddsr_description/urdf/ddsr.xacro (robot description, xacro)
@@ -16,6 +16,6 @@
 <!-- user input dimensions  ( DEBUG: all mass values have been divided by 100 )  -->
 <xacro:property name="robot" value="ddsr" />
-<xacro:property name="base_length" value="1.0" />
-<xacro:property name="base_width" value="0.5" />
+<xacro:property name="base_length" value="0.8" />
+<xacro:property name="base_width" value="0.6" />
 <xacro:property name="base_height" value="0.2" />
 <xacro:property name="base_mass" value="300.0" />
@@ -55,10 +55,10 @@
 </link>
 <!-- Base Link. STL is scaled with te ratio between NEW/OLD dimensions -->
-<joint name="$footprint_2_base" type="fixed" >
+<joint name="$footprint_2_platform" type="fixed" >
 	<parent link="footprint"/>
-	<child link="base"/>
-	<origin xyz="0 0 ${floor_clearance+base_height*0.5}" rpy="0 0 0"/>
-</joint>
-<link name="base">
+	<child link="platform"/>
+	<origin xyz="${base_length*0.25} 0 ${floor_clearance+base_height*0.5}" rpy="0 0 0"/>
+</joint>
+<link name="platform">
 	<visual>
 		<origin xyz="0 0 0" rpy="0 0 0"/>
@@ -86,8 +86,8 @@
 </link>
 <!-- ~~~~~~~~~~~~~~~~~~~~~~~ DRIVE WHEELS ~~~~~~~~~~~~~~~~~~~~~~~~~~~~~~~~~~~~~~~~ -->
-<joint name="$base_2_left_wheel" type="continuous" >
-	<parent link="base"/>
+<joint name="$platform_2_left_wheel" type="continuous" >
+	<parent link="platform"/>
 	<child link="left_wheel"/>
-	<origin xyz="${-base_length*0.25} ${base_width*0.5} ${-base_height*0.5+wheel_radius-floor_clearance}" rpy="${-0.5*pi} 0 0"/>
+	<origin xyz="${-base_length*0.3} ${base_width*0.5} ${-base_height*0.5+wheel_radius-floor_clearance}" rpy="${-0.5*pi} 0 0"/>
 	<axis xyz="0 0 1"/>
 	<limit effort="99999" velocity="${20*pi}"/>
@@ -119,8 +119,8 @@
 	</inertial>
 </link>
-<joint name="$base_2_right_wheel" type="continuous" >
-	<parent link="base"/>
+<joint name="$platform_2_right_wheel" type="continuous" >
+	<parent link="platform"/>
 	<child link="right_wheel"/>
-	<origin xyz="${-base_length*0.25} ${-base_width*0.5} ${-base_height*0.5+wheel_radius-floor_clearance}" rpy="${0.5*pi} 0 0"/>
+	<origin xyz="${-base_length*0.3} ${-base_width*0.5} ${-base_height*0.5+wheel_radius-floor_clearance}" rpy="${0.5*pi} 0 0"/>
 	<axis xyz="0 0 1"/>
 	<limit effort="99999" velocity="${20*pi}"/>
@@ -153,8 +153,8 @@
 </link>
 <!-- ~~~~~~~~~~~~~~~~~~~~~~~ CASTER WHEEL ~~~~~~~~~~~~~~~~~~~~~~~~~~~~~~~~~~~~~~~~ -->
-<joint name="$base_2_caster_hinge_1" type="continuous" >
-	<parent link="base"/>
+<joint name="$platform_2_caster_hinge_1" type="continuous" >
+	<parent link="platform"/>
 	<child link="caster_hinge_1"/>
-	<origin xyz="${base_length*0.4} 0 ${-base_height*0.5-0.02}" rpy="0 0 0"/>
+	<origin xyz="${base_length*0.4} 0 ${-base_height*0.5-0.01}" rpy="0 0 0"/>
 	<axis xyz="0 0 1"/>
 	<limit effort="100000." velocity="${2*pi}"/>
@@ -165,5 +165,5 @@
 		<origin xyz="0 0 0" rpy="0 0 0"/>
 		<geometry>
-			<box size="0.02 0.02 0.04"/>
+			<box size="0.02 0.02 0.02"/>
 		</geometry>
 		<material name="ddsr/red" />
@@ -172,5 +172,5 @@
 		<origin xyz="0 0 0" rpy="0 0 0"/>
 		<geometry>
-			<box size="0.02 0.02 0.04"/>
+			<box size="0.02 0.02 0.02"/>
 		</geometry>
 	</collision>
@@ -178,8 +178,8 @@
 		<mass value="1" />
 		<origin xyz="0 0 0" rpy="0 0 0"/>
-		<inertia ixx="${0.083*(0.02*0.02+0.04*0.04)}"
-			ixy="0.0"
-			ixz="0.0"
-			iyy="${0.083*(0.02*0.02+0.04*0.04)}"
+		<inertia ixx="${0.083*(0.02*0.02+0.02*0.02)}"
+			ixy="0.0"
+			ixz="0.0"
+			iyy="${0.083*(0.02*0.02+0.02*0.02)}"
 			iyz="0.0"
 			izz="${0.083*(0.02*0.02+0.02*0.02)}" />
@@ -189,5 +189,5 @@
 	<parent link="caster_hinge_1"/>
 	<child link="caster_hinge_2"/>
-	<origin xyz="${-0.04*0.707*0.5} 0 ${-0.02-0.04*0.707*0.5}" rpy="0 ${0.25*pi} 0"/>
+	<origin xyz="${-0.04*0.707*0.5} 0 ${-0.01-0.04*0.707*0.5}" rpy="0 ${0.25*pi} 0"/>
 </joint>
 <link name="caster_hinge_2">
@@ -216,3 +216,36 @@
 	</inertial>
 </link>
+<joint name="$caster_hinge_2_2_caster_wheel" type="continuous" >
+	<parent link="caster_hinge_2"/>
+	<child link="caster_wheel"/>
+	<origin xyz="0 0 ${-0.04*0.707*0.5}" rpy="-${0.5*pi} 0 0"/>
+	<axis xyz="0 0 1"/>
+	<limit effort="99999" velocity="${20*pi}"/>
+	<dynamics friction="0.25" damping="0.05"/>
+</joint>
+<link name="caster_wheel">
+	<visual>
+		<origin xyz="0 0 0" rpy="0 0 0"/>
+		<geometry>
+			<cylinder length="${0.5*wheel_width}" radius="${floor_clearance-0.02-0.04*0.707}"/>
+		</geometry>
+		<material name="ddsr/grey" />
+	</visual>
+	<collision>
+		<origin xyz="0 0 0" rpy="0 0 0"/>
+		<geometry>
+			<cylinder length="${0.5*wheel_width}" radius="${floor_clearance-0.02-0.04*0.707}"/>
+		</geometry>
+	</collision>
+	<inertial>
+		<mass value="${wheel_mass*0.5}" />
+		<origin xyz="0 0 0" rpy="0 0 0"/>
+		<inertia ixx="${0.083*wheel_mass*0.5*(3*wheel_radius*wheel_radius+wheel_width*wheel_width)}"
+			ixy="0.0"
+			ixz="0.0"
+			iyy="${0.083*wheel_mass*0.5*(3*wheel_radius*wheel_radius+wheel_width*wheel_width)}"
+			iyz="0.0"
+			izz="${0.5*wheel_mass*0.5*wheel_radius*wheel_radius}" />
+	</inertial>
+</link>
 </robot>

Commit message: Added transmissions at description

File: ddsr_description/urdf/ddsr.xacro (robot description, xacro)
@@ -42,6 +42,6 @@
 </material>
 <!-- Extra definitions for gazebo simulation  -->
-<!-- <xacro:include filename="$(find rob1500_gazebo)/gazebo/rob1500.gazebo" /> -->
-<!-- <xacro:gazebo_include gazebo_namespace="$(arg namespace)" /> -->
+<xacro:include filename="$(find ddsr_gazebo)/gazebo/ddsr.gazebo" />
+<xacro:gazebo_include gazebo_namespace="$(arg namespace)" />
 <!-- ~~~~~~~~~~~~~~~~~~~~~~~ PLATFORM ~~~~~~~~~~~~~~~~~~~~~~~~~~~~~~~~~~~~~~~~ -->
 <link name="footprint">
@@ -152,6 +152,26 @@
 	</inertial>
 </link>
+<transmission name="$platform_2_left_wheel_transmission">
+	<type>transmission_interface/SimpleTransmission</type>
+	<joint name="platform_2_left_wheel">
+		<hardwareInterface>hardware_interface/VelocityJointInterface</hardwareInterface>
+	</joint>
+	<actuator name="left_wheel_motor">
+		<hardwareInterface>EffortJointInterface</hardwareInterface>
+		<mechanicalReduction>30</mechanicalReduction>
+	</actuator>
+</transmission>
+<transmission name="$platform_2_right_wheel_transmission">
+	<type>transmission_interface/SimpleTransmission</type>
+	<joint name="platform_2_right_wheel">
+		<hardwareInterface>hardware_interface/VelocityJointInterface</hardwareInterface>
+	</joint>
+	<actuator name="right_wheel_motor">
+		<hardwareInterface>EffortJointInterface</hardwareInterface>
+		<mechanicalReduction>30</mechanicalReduction>
+	</actuator>
+</transmission>
 <!-- ~~~~~~~~~~~~~~~~~~~~~~~ CASTER WHEEL ~~~~~~~~~~~~~~~~~~~~~~~~~~~~~~~~~~~~~~~~ -->
-<joint name="$platform_2_caster_hinge_1" type="continuous" >
+<joint name="platform_2_caster_hinge_1" type="continuous" >
 	<parent link="platform"/>
 	<child link="caster_hinge_1"/>
@@ -186,5 +206,5 @@
 	</inertial>
 </link>
-<joint name="$caster_hinge_1_2_caster_hinge_2" type="fixed" >
+<joint name="caster_hinge_1_2_caster_hinge_2" type="fixed" >
 	<parent link="caster_hinge_1"/>
 	<child link="caster_hinge_2"/>
@@ -216,5 +236,5 @@
 	</inertial>
 </link>
-<joint name="$caster_hinge_2_2_caster_wheel" type="continuous" >
+<joint name="caster_hinge_2_2_caster_wheel" type="continuous" >
 	<parent link="caster_hinge_2"/>
 	<child link="caster_wheel"/>
@@ -249,3 +269,23 @@
 	</inertial>
 </link>
+<!--  caster steering free transmission -->
+<transmission name="platform_2_caster_hinge_1_transmission">
+	<type>transmission_interface/SimpleTransmission</type>
+	<joint name="platform_2_caster_hinge_1">
+		<hardwareInterface>hardware_interface/EffortJointInterface</hardwareInterface>
+	</joint>
+	<actuator name="platform_2_caster_hinge_1_steering">
+		<mechanicalReduction>1</mechanicalReduction>
+	</actuator>
+</transmission>
+<!-- caster drive free transmission -->
+<transmission name="caster_hinge_2_2_caster_wheel_transmission">
+	<type>transmission_interface/SimpleTransmission</type>
+	<joint name="caster_hinge_2_2_caster_wheel">
+		<hardwareInterface>hardware_interface/EffortJointInterface</hardwareInterface>
+	</joint>
+	<actuator name="caster_hinge_2_2_caster_driving">
+		<mechanicalReduction>1</mechanicalReduction>
+	</actuator>
+</transmission>
 </robot>

Commit message: Fixed bug at joint name

File: ddsr_description/urdf/ddsr.xacro (robot description, xacro)
@@ -86,5 +86,5 @@
 </link>
 <!-- ~~~~~~~~~~~~~~~~~~~~~~~ DRIVE WHEELS ~~~~~~~~~~~~~~~~~~~~~~~~~~~~~~~~~~~~~~~~ -->
-<joint name="$platform_2_left_wheel" type="continuous" >
+<joint name="platform_2_left_wheel" type="continuous" >
 	<parent link="platform"/>
 	<child link="left_wheel"/>
@@ -119,5 +119,5 @@
 	</inertial>
 </link>
-<joint name="$platform_2_right_wheel" type="continuous" >
+<joint name="platform_2_right_wheel" type="continuous" >
 	<parent link="platform"/>
 	<child link="right_wheel"/>

Commit message: Diff drive controller working fine. Added control rviz with odometry pose list.

File: ddsr_description/urdf/ddsr.xacro (robot description, xacro)
@@ -122,5 +122,5 @@
 	<parent link="platform"/>
 	<child link="right_wheel"/>
-	<origin xyz="${-base_length*0.3} ${-base_width*0.5} ${-base_height*0.5+wheel_radius-floor_clearance}" rpy="${0.5*pi} 0 0"/>
+	<origin xyz="${-base_length*0.3} ${-base_width*0.5} ${-base_height*0.5+wheel_radius-floor_clearance}" rpy="${-0.5*pi} 0 0"/>
 	<axis xyz="0 0 1"/>
 	<limit effort="99999" velocity="${20*pi}"/>

Commit message: Added teleop launch with mouse teleop joy

File: ddsr_description/urdf/ddsr.xacro (robot description, xacro)
@@ -91,5 +91,5 @@
 	<origin xyz="${-base_length*0.3} ${base_width*0.5} ${-base_height*0.5+wheel_radius-floor_clearance}" rpy="${-0.5*pi} 0 0"/>
 	<axis xyz="0 0 1"/>
-	<limit effort="99999" velocity="${20*pi}"/>
+	<limit effort="10" velocity="${20*pi}"/>
 	<dynamics friction="0.25" damping="0.05"/>
 </joint>

Commit message: Added front lidar and gazebo lidar plugin

File: ddsr_description/urdf/ddsr.xacro (robot description, xacro)
@@ -85,4 +85,35 @@
 	</inertial>
 </link>
+<!-- Base Link. STL is scaled with te ratio between NEW/OLD dimensions -->
+<joint name="$platform_2_lidar" type="fixed" >
+	<parent link="platform"/>
+	<child link="lidar"/>
+	<origin xyz="${base_length*0.4} 0 ${base_height*0.6}" rpy="0 0 0"/>
+</joint>
+<link name="lidar">
+	<visual>
+		<origin xyz="0 0 0" rpy="0 0 0"/>
+		<geometry>
+			<box size="0.1 0.1 0.1"/>
+		</geometry>
+		<material name="ddsr/red" />
+	</visual>
+	<collision>
+		<origin xyz="0 0 0" rpy="0 0 0"/>
+		<geometry>
+			<box size="0.1 0.1 0.1"/>
+		</geometry>
+	</collision>
+	<inertial>
+		<mass value="1.0" />
+		<origin xyz="0 0 0" rpy="0 0 0"/>
+		<inertia ixx="${0.083*1*(0.1*0.1+0.1*0.1)}"
+			ixy="0.0"
+			ixz="0.0"
+			iyy="${0.083*1*(0.1*0.1+0.1*0.1)}"
+			iyz="0.0"
+			izz="${0.083*1*(0.1*0.1+0.1*0.1)}" />
+	</inertial>
+</link>
 <!-- ~~~~~~~~~~~~~~~~~~~~~~~ DRIVE WHEELS ~~~~~~~~~~~~~~~~~~~~~~~~~~~~~~~~~~~~~~~~ -->
 <joint name="platform_2_left_wheel" type="continuous" >
